Commit message: initial

File: Week1/Challenge/motor_sim/urdf/dc_motor.urdf (robot description, URDF)
Before this commit: robot dc_motor, 3 links, 2 joints
Links:
- link Motor: geometry visual mesh filename=package://motor_sim/models/dcMotor.stl
- link Wheel: geometry visual mesh filename=package://motor_sim/models/MCR2_1000_1_1_Wheel_Coupler_2.stl
Joints:
- joint joint1: child (none) -> Motor; origin (none) -> xyz=0 0 1 rpy=0 0 0; parent (none) -> world
- joint joint2: axis (none) -> 1 0 0; child (none) -> Wheel; origin (none) -> xyz=0.041475 0 0 rpy=0 0 0; parent (none) -> Motor
